File: Hard/Motion.sch (KiCad schematic (older format))
At the start: 54 parts, among them J2 KRC_Conn_SWD, J3 USB_B_Micro, J4 KRC_Conn_CAN, U1 CY8C58xxLTI-LPxxx, U2 W25N01GVxxIG-IT, U3 NCV7342, U4 BMI088, Y1 24MHz

Commit message: [update] READMEを整備
Parts:
- D4, D5: Agency 秋月電子 -> akizuki
- U4: Agency (none) -> Digikey; Link (none) -> https://www.digikey.jp/product-detail/ja/bosch-sensortec/BM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; MPN (none) -> BMI088
Changed lines of the file:
@@
 EESchema Schematic File Version 4
+LIBS:Motion-cache
 EELAYER 26 0
 EELAYER END
@@
 F 2 "Diode_SMD:D_TUMD2" V 2250 750 50  0001 C CNN
 F 3 "http://akizukidenshi.com/download/ds/rohm/rsx101vam30-j.pdf" V 2250 750 50  0001 C CNN
-F 4 "秋月電子" H 2250 750 50  0001 C CNN "Agency"
+F 4 "akizuki" H 2250 750 50  0001 C CNN "Agency"
 F 5 "http://akizukidenshi.com/catalog/g/gI-05951/" H 2250 750 50  0001 C CNN "Link"
 F 6 "RSX101VAM-30TR" H 2250 750 50  0001 C CNN "MPN"
@@
 F 2 "Diode_SMD:D_TUMD2" V 2250 1800 50  0001 C CNN
 F 3 "http://akizukidenshi.com/download/ds/rohm/rsx101vam30-j.pdf" V 2250 1800 50  0001 C CNN
-F 4 "秋月電子" H 2250 1800 50  0001 C CNN "Agency"
+F 4 "akizuki" H 2250 1800 50  0001 C CNN "Agency"
 F 5 "http://akizukidenshi.com/catalog/g/gI-05951/" H 2250 1800 50  0001 C CNN "Link"
 F 6 "RSX101VAM-30TR" H 2250 1800 50  0001 C CNN "MPN"
@@
 F 2 "KUTKiCad_footprint:Bosch_QFN-16_4.5x3.0mm_P0.5mm_Handsoldering" H 5700 8150 50  0001 C CNN
 F 3 "https://ae-bst.resource.bosch.com/media/_tech/media/datasheets/BST-BMI088-DS001.pdf" H 5700 8150 50  0001 C CNN
+F 4 "Digikey" H 5700 7000 50  0001 C CNN "Agency"
+F 5 "BMI088" H 5700 7000 50  0001 C CNN "MPN"
+F 6 "https://www.digikey.jp/product-detail/ja/bosch-sensortec/BMI088/828-1082-1-ND/8634942" H 5700 7000 50  0001 C CNN "Link"
 	1    5700 7000
 	1    0    0    -1
